File: hardware/kicad/cc1101-morse/cc1101-morse.kicad_pcb (KiCad board)
At the start: 2 copper layers, 40 x 60 mm, 12 parts, among them J1 Conn_02x04_Odd_Even, SW1 SW_Push, U1 ESP32-C3-SuperMini

Commit message: Adding vinilabs.cc
Other:
- board text added: "vinilabs.cc"
Changed lines of the file:
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@@
 		(layer "Edge.Cuts")
+	)
+	(gr_text "vinilabs.cc"
+		(at 145 129 0)
+		(layer "F.SilkS")
+		(effects
+			(font
+				(size 1 1)
+				(thickness 0.1)
+			)
+			(justify left bottom)
+		)
 	)
 	(segment
@@
 	)
 	(segment
+		(start 146 92)
+		(end 143.5 89.5)
+		(width 0.4)
+		(layer "F.Cu")
+		(net "+3V3")
+	)
+	(segment
+		(start 143.5 77)
+		(end 144.5 76)
+		(width 0.4)
+		(layer "F.Cu")
+		(net "+3V3")
+	)
+	(segment
+		(start 143.5 89.5)
+		(end 143.5 77)
+		(width 0.4)
+		(layer "F.Cu")
+		(net "+3V3")
+	)
+	(segment
+		(start 146.19 95.88)
+		(end 146.19 92.19)
+		(width 0.4)
+		(layer "F.Cu")
+		(net "+3V3")
+	)
+	(segment
+		(start 146.19 92.19)
+		(end 146 92)
+		(width 0.4)
+		(layer "F.Cu")
+		(net "+3V3")
+	)
+	(segment
+		(start 144.5 76)
+		(end 145.88 76)
+		(width 0.4)
+		(layer "F.Cu")
+		(net "+3V3")
+	)
+	(segment
 		(start 139 90)
 		(end 139 85)
@@
 		(net "Net-(J1-Pin_6)")
 	)
-	(segment
-		(start 146 92)
-		(end 143.5 89.5)
-		(width 0.4)
-		(layer "F.Cu")
-		(net "+3V3")
-	)
-	(segment
-		(start 143.5 77)
-		(end 144.5 76)
-		(width 0.4)
-		(layer "F.Cu")
-		(net "+3V3")
-	)
-	(segment
-		(start 143.5 89.5)
-		(end 143.5 77)
-		(width 0.4)
-		(layer "F.Cu")
-		(net "+3V3")
-	)
-	(segment
-		(start 146.19 95.88)
-		(end 146.19 92.19)
-		(width 0.4)
-		(layer "F.Cu")
-		(net "+3V3")
-	)
-	(segment
-		(start 146.19 92.19)
-		(end 146 92)
-		(width 0.4)
-		(layer "F.Cu")
-		(net "+3V3")
-	)
-	(segment
-		(start 144.5 76)
-		(end 145.88 76)
-		(width 0.4)
-		(layer "F.Cu")
-		(net "+3V3")
-	)
 	(zone

Commit message: Fix the CC1101 socket pinout to match the module
J1 now carries the module's own order: GND, VCC, GDO0, CSN, SCK,
MOSI, MISO, GDO2.

Two things were wrong before. The supply pair was reversed — pad 1
was +3V3 where the module has GND — so plugging a module into the
board would have applied power backwards across it. And all six
signals were offset, so nothing would have talked even had the module
survived.

Caught on the breadboard: status reported PARTNUM 0xFF VERSION 0xFF,
MISO stuck high, which is what a module that is not driving the bus
looks like.

The signals cost nothing to fix. Every SPI line here is bit-banged,
so no pin is special — radio.h just renames which GPIO is which
function, six #defines, no re-routing. Power was the exception: rails
are physical and that pair had to be corrected on the board.

DRC: 0 unconnected, 0 parity. The one remaining violation is a
footprint/library mismatch warning, expected after editing the
footprint's pad numbering.

Firmware compiles clean at 27% flash.
Parts:
- added J2: Conn_01x02_Socket, Connector_PinSocket_2.54mm:PinSocket_1x02_P2.54mm_Vertical, F.Cu at (135.5, 107.5)
- added J3: Conn_01x02_Socket, Connector_PinSocket_2.54mm:PinSocket_1x02_P2.54mm_Vertical, F.Cu at (138.5, 119.0)
Connections:
- J1 pad 1: +3V3 -> GND
- J1 pad 2: GND -> +3V3
- U1 pad 1: Net-(J1-Pin_7) -> Net-(J1-Pin_8)
- U1 pad 10: Net-(J1-Pin_3) -> Net-(J1-Pin_4)
- U1 pad 11: Net-(J1-Pin_6) -> Net-(J1-Pin_5)
- U1 pad 12: unconnected-(U1-GPIO8-Pad12) -> Net-(J3-Pin_2)
- U1 pad 13: unconnected-(U1-GPIO9-Pad13) -> Net-(J3-Pin_1)
- U1 pad 2: Net-(J1-Pin_8) -> Net-(J1-Pin_7)
- U1 pad 3: Net-(J1-Pin_5) -> Net-(J1-Pin_6)
- U1 pad 9: Net-(J1-Pin_4) -> Net-(J1-Pin_3)
Routing:
- net Net-(J1-Pin_6): track 35.9 -> 73.4 mm
- net Net-(J1-Pin_5): track 73.4 -> 35.9 mm
- net Net-(J1-Pin_4): track 36.8 -> 63.8 mm
- net Net-(J1-Pin_3): track 60.3 -> 36.8 mm
- net Net-(J3-Pin_1): track 0.00 -> 18.1 mm
- net +3V3: track 22.8 -> 37.3 mm
- net Net-(J3-Pin_2): track 0.00 -> 11.3 mm
- net Net-(J1-Pin_8): track 18.5 -> 22.1 mm
- net Net-(J1-Pin_7): track 22.1 -> 18.5 mm
