File: hardware/kicad/cc1101-morse/cc1101-morse.kicad_pcb (KiCad board)
At the start: 2 copper layers, 40 x 60 mm, 15 parts, among them J1 Conn_02x04_Odd_Even, J2 Conn_01x04_Socket, SW1 SW_Push, U1 ESP32-C3-SuperMini

Commit message: Tidy the board; refresh the renders
Removes a 0.06 mm +3V3 fragment left behind by an earlier track
split. Electrically nothing, but DRC flagged it as a dangling end and
the laser would have etched it as a copper spur.

Schematic changed too, though its netlist is byte-identical — the
edit was cosmetic. All three renders regenerated.

DRC back to the three documented exceptions: the TP4/U1 courtyard
overlap, the J1 footprint/library mismatch, and +3V3 arriving in two
pieces because the TP3-TP4 link is off-board.

84 segments, 76 at 0.6 mm and 8 at 0.4 mm past U1's pads. Exports
regenerated; 46 holes.
Parts:
- TP3, TP4: value TestPoint -> +3V3

Commit message: Changing ESP32 pad shapes from circular to oval to improve etching
Routing:
- net Net-(J1-Pin_6): track 72.3 -> 72.9 mm
Changed lines of the file:
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@@
 			(layer "F.Fab")
 		)
-		(pad "1" thru_hole circle
+		(pad "1" thru_hole oval
 			(at 7.62 8.89 90)
-			(size 1.14 1.14)
+			(size 2 1.14)
 			(drill 0.84)
 			(layers "*.Cu" "*.Mask")
@@
 			(pintype "bidirectional")
 		)
-		(pad "2" thru_hole circle
+		(pad "2" thru_hole oval
 			(at 7.62 6.35 90)
-			(size 1.14 1.14)
+			(size 2 1.14)
 			(drill 0.84)
 			(layers "*.Cu" "*.Mask")
@@
 			(pintype "bidirectional")
 		)
-		(pad "3" thru_hole circle
+		(pad "3" thru_hole oval
 			(at 7.62 3.81 90)
-			(size 1.14 1.14)
+			(size 2 1.14)
 			(drill 0.84)
 			(layers "*.Cu" "*.Mask")
@@
 			(pintype "bidirectional+no_connect")
 		)
-		(pad "6" thru_hole circle
+		(pad "6" thru_hole oval
 			(at 7.62 -3.81 90)
-			(size 1.14 1.14)
+			(size 2 1.14)
 			(drill 0.84)
 			(layers "*.Cu" "*.Mask")
@@
 			(pintype "power_in")
 		)
-		(pad "8" thru_hole circle
+		(pad "8" thru_hole oval
 			(at 7.62 -8.89 90)
-			(size 1.14 1.14)
+			(size 2 1.14)
 			(drill 0.84)
 			(layers "*.Cu" "*.Mask")
@@
 			(pintype "power_in")
 		)
-		(pad "9" thru_hole circle
+		(pad "9" thru_hole oval
 			(at -7.62 -8.89 90)
-			(size 1.14 1.14)
+			(size 2 1.14)
 			(drill 0.84)
 			(layers "*.Cu" "*.Mask")
@@
 			(pintype "bidirectional")
 		)
-		(pad "10" thru_hole circle
+		(pad "10" thru_hole oval
 			(at -7.62 -6.35 90)
-			(size 1.14 1.14)
+			(size 2 1.14)
 			(drill 0.84)
 			(layers "*.Cu" "*.Mask")
@@
 			(pintype "bidirectional")
 		)
-		(pad "11" thru_hole circle
+		(pad "11" thru_hole oval
 			(at -7.62 -3.81 90)
-			(size 1.14 1.14)
+			(size 2 1.14)
 			(drill 0.84)
 			(layers "*.Cu" "*.Mask")
@@
 			(pintype "bidirectional")
 		)
-		(pad "12" thru_hole circle
+		(pad "12" thru_hole oval
 			(at -7.62 -1.27 90)
-			(size 1.14 1.14)
+			(size 2 1.14)
 			(drill 0.84)
 			(layers "*.Cu" "*.Mask")
@@
 			(pintype "bidirectional")
 		)
-		(pad "13" thru_hole circle
+		(pad "13" thru_hole oval
 			(at -7.62 1.27 90)
-			(size 1.14 1.14)
+			(size 2 1.14)
 			(drill 0.84)
 			(layers "*.Cu" "*.Mask")
@@
 			(pintype "bidirectional")
 		)
-		(pad "14" thru_hole circle
+		(pad "14" thru_hole oval
 			(at -7.62 3.81 90)
-			(size 1.14 1.14)
+			(size 2 1.14)
 			(drill 0.84)
 			(layers "*.Cu" "*.Mask")
@@
 			(pintype "bidirectional")
 		)
-		(pad "15" thru_hole circle
+		(pad "15" thru_hole oval
 			(at -7.62 6.35 90)
-			(size 1.14 1.14)
+			(size 2 1.14)
 			(drill 0.84)
 			(layers "*.Cu" "*.Mask")
@@
 	)
 	(segment
+		(start 162.5 79.5)
+		(end 156.5 73.5)
+		(width 0.6)
+		(layer "B.Cu")
+		(net "Net-(J1-Pin_6)")
+	)
+	(segment
 		(start 155.08 98.58)
 		(end 153.81 97.31)
@@
 	)
 	(segment
-		(start 152.04 73.5)
-		(end 156.5 73.5)
-		(width 0.6)
-		(layer "B.Cu")
-		(net "Net-(J1-Pin_6)")
-	)
-	(segment
 		(start 153.81 97.31)
 		(end 153.81 95.88)
@@
 	)
 	(segment
-		(start 150.96 76)
+		(start 155.08 111.93463)
+		(end 155.08 108.58)
+		(width 0.4)
+		(layer "B.Cu")
+		(net "Net-(J1-Pin_6)")
+	)
+	(segment
+		(start 156.433948 113)
+		(end 156.14537 113)
+		(width 0.4)
+		(layer "B.Cu")
+		(net "Net-(J1-Pin_6)")
+	)
+	(segment
+		(start 160 113.5)
+		(end 162.5 111)
+		(width 0.6)
+		(layer "B.Cu")
+		(net "Net-(J1-Pin_6)")
+	)
+	(segment
+		(start 156.433948 113)
+		(end 156.933948 113.5)
+		(width 0.6)
+		(layer "B.Cu")
+		(net "Net-(J1-Pin_6)")
+	)
+	(segment
+		(start 152.04 73.5)
 		(end 150.96 74.58)
 		(width 0.6)
@@
 	)
 	(segment
-		(start 160.5 113)
-		(end 156.433948 113)
-		(width 0.6)
-		(layer "B.Cu")
-		(net "Net-(J1-Pin_6)")
-	)
-	(segment
-		(start 155.08 108.58)
-		(end 155.08 111.646052)
+		(start 156.14537 113)
+		(end 155.08 111.93463)
 		(width 0.4)
 		(layer "B.Cu")
@@
 	)
 	(segment
+		(start 156.933948 113.5)
+		(end 160 113.5)
+		(width 0.6)
+		(layer "B.Cu")
+		(net "Net-(J1-Pin_6)")
+	)
+	(segment
 		(start 156.5 73.5)
-		(end 162.5 79.5)
+		(end 152.04 73.5)
 		(width 0.6)
 		(layer "B.Cu")
@@
 	(segment
 		(start 150.96 74.58)
-		(end 152.04 73.5)
-		(width 0.6)
-		(layer "B.Cu")
-		(net "Net-(J1-Pin_6)")
-	)
-	(segment
-		(start 162.5 111)
-		(end 160.5 113)
-		(width 0.6)
-		(layer "B.Cu")
-		(net "Net-(J1-Pin_6)")
-	)
-	(segment
-		(start 162.5 79.5)
-		(end 162.5 111)
+		(end 150.96 76)
 		(width 0.6)
 		(layer "B.Cu")
@@
 	)
 	(segment
-		(start 156.433948 113)
-		(end 155.08 111.646052)
-		(width 0.4)
-		(layer "B.Cu")
-		(net "Net-(J1-Pin_6)")
+		(start 162.5 111)
+		(end 162.5 79.5)
+		(width 0.6)
+		(layer "B.Cu")
+		(net "Net-(J1-Pin_6)")
