File: hardware/kicad/cc1101-morse/cc1101-morse.kicad_sch (KiCad schematic)
At the start: 11 parts, among them J1 Conn_02x04_Odd_Even, J2 Conn_01x04_Socket, SW1 SW_Push, U1 ESP32-C3-SuperMini

Commit message: Tidy the board; refresh the renders
Removes a 0.06 mm +3V3 fragment left behind by an earlier track
split. Electrically nothing, but DRC flagged it as a dangling end and
the laser would have etched it as a copper spur.

Schematic changed too, though its netlist is byte-identical — the
edit was cosmetic. All three renders regenerated.

DRC back to the three documented exceptions: the TP4/U1 courtyard
overlap, the J1 footprint/library mismatch, and +3V3 arriving in two
pieces because the TP3-TP4 link is off-board.

84 segments, 76 at 0.6 mm and 8 at 0.4 mm past U1's pads. Exports
regenerated; 46 holes.
Parts:
- TP3, TP4: value TestPoint -> +3V3
Changed lines of the file:
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@@
 			)
 		)
-		(property "Value" "TestPoint"
+		(property "Value" "+3V3"
 			(at 100.33 109.9821 0)
 			(hide yes)
@@
 			)
 		)
-		(property "Value" "TestPoint"
+		(property "Value" "+3V3"
 			(at 88.9 109.9821 0)
 			(hide yes)
