File: hardware/kicad/cc1101-morse/cc1101-morse.kicad_sch (KiCad schematic)
At the start: 11 parts, among them J1 Conn_02x04_Odd_Even, J2 Conn_01x04_Socket, SW1 SW_Push, U1 ESP32-C3-SuperMini

Commit message: .
Parts:
- J2: footprint Connector_PinSocket_2.54mm:PinSocket_1x04_P2.54mm_Vertical -> Connector_JST:JST_XH_B4B-XH-A_1x04_P2.50mm_Vertical
Changed lines of the file:
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@@
 			)
 		)
-		(property "Footprint" "Connector_PinSocket_2.54mm:PinSocket_1x04_P2.54mm_Vertical"
+		(property "Footprint" "Connector_JST:JST_XH_B4B-XH-A_1x04_P2.50mm_Vertical"
 			(at 128.27 59.69 0)
 			(hide yes)
